File: NXP/KiCAD/Buttons/Sparkfun_buttons/Sparkfun_buttons.sch (KiCad schematic (older format))
At the start: 2 parts

Commit message: did some schematic work on the buttons. Still lots todo. Added todo to nxp/kicad/readme
Parts:
- removed SW?: 15mm_Silicone_Buttons, symbol SF_~COM_07835:15mm_Silicone_Buttons
- added D1, D2, D3, D4, D5, D6, D7, D8: LED_RGBC, symbol Device:LED_RGBC
- added R1, R10, R11, R12, R13, R14, R15, R16, R17, R18, R19, R2, R20, R21, R22, R23, R24, R3, R4, R5, R6, R7, R8, R9: R_Small_US, symbol Device:R_Small_US
- added RN1, RN2: R_Pack04, symbol Device:R_Pack04
- added SW2: 15mm_Silicone_Buttons, symbol SF_~COM_07835:15mm_Silicone_Buttons
- gave numbers to parts that had none: 1
Connections:
- net labels added: B1, B2, B3, B4
- wire segments 34 -> 98

Commit message: working on keyboard. Made symbol for stock 596 shift register.
Parts:
- added U? (x3): 596A_8bit_Shift_Register, symbol NPIC6C596A:596A_8bit_Shift_Register
Connections:
- net labels added: Blue_0, Blue_1, Blue_2, Blue_3, Blue_4, Blue_5, Blue_6, Blue_7, Blue_Data, Blue_Serial_Out, Green_0, Green_1, Green_2, Green_3, Green_4, Green_5, Green_6, Green_7, Green_Data, Green_Serial_Out, Red_0, Red_1, Red_2, Red_3, Red_4, Red_5, Red_6, Red_7, Red_Data, Red_Serial_Out, Shift_Clk, Storage_Clk, ~Output, ~RESET
- wire segments 98 -> 146

Commit message: made symbol from data controlled LEDs from liteon. Will cut down on hardware costs.
Parts:
- removed D1, D2, D3, D4, D5, D6, D7, D8: LED_RGBC, symbol Device:LED_RGBC
- removed R1, R10, R11, R12, R13, R14, R15, R16, R17, R18, R19, R2, R20, R21, R22, R23, R24, R3, R4, R5, R6, R7, R8, R9: R_Small_US, symbol Device:R_Small_US
- removed U? (x3): 596A_8bit_Shift_Register, symbol NPIC6C596A:596A_8bit_Shift_Register
- added D? (x8): LTST-E563CEGBW, symbol liteon:LTST-E563CEGBW
Connections:
- net labels removed: Blue_0, Blue_1, Blue_2, Blue_3, Blue_4, Blue_5, Blue_6, Blue_7, Blue_Data, Blue_Serial_Out, Green_0, Green_1, Green_2, Green_3, Green_4, Green_5, Green_6, Green_7, Green_Data, Green_Serial_Out, Red_0, Red_1, Red_2, Red_3, Red_4, Red_5, Red_6, Red_7, Red_Data, Red_Serial_Out, Shift_Clk, Storage_Clk, ~Output, ~RESET
- wire segments 146 -> 58

Commit message: WIP button board with initial layout ready for review.
Parts:
- removed D? (x7): LTST-E563CEGBW, symbol liteon:LTST-E563CEGBW
- removed SW2: 15mm_Silicone_Buttons, symbol SF_~COM_07835:15mm_Silicone_Buttons
- added C1, C2, C3, C4, C5, C6, C7, C8: 0.1uF, Capacitor_SMD:C_0805_2012Metric_Pad1.15x1.40mm_HandSolder, symbol Device:C_Small
- added D2, D3, D4, D5, D6, D7, D8: LTST-E563CEGBW, liteon:LTST-E563CEGBW_RGB_LED_4pad_5x4, symbol liteon:LTST-E563CEGBW
- added H1, H2, H3: MountingHole, MountingHole:MountingHole_3.2mm_M3, symbol Mechanical:MountingHole
- added J1: Screw_Terminal_01x12, TerminalBlock_RND:TerminalBlock_RND_205-00022_1x12_P5.00mm_Horizontal, symbol Connector:Screw_Terminal_01x12
- added RN3, RN4: R_Pack04, Resistor_SMD:R_Array_Convex_4x0603, symbol Device:R_Pack04
- D1: renamed from D?; footprint (none) -> liteon:LTST-E563CEGBW_RGB_LED_4pad_5x4
- RN1, RN2: footprint (none) -> Resistor_SMD:R_Array_Convex_4x0603
- SW1: footprint (none) -> Sparkfun_buttons:SF_ COM_07835
Connections:
- net labels added: +5V, B5, B6, B7, B8, Dcon, Din, Dout, GND, Vcc
- net labels removed: +3V3
- wire segments 58 -> 137
Other:
- moved on the sheet: RN1, RN2
