File: NXP/KiCAD/joystick/joystick.sch (KiCad schematic (older format))
At the start: 7 parts, among them J1 Screw_Terminal_01x05

Commit message: Finished joystick design and layout.
Parts:
- H1, H2, H3, H4: footprint (none) -> MountingHole:MountingHole_3.2mm_M3
- J1: footprint (none) -> TerminalBlock_RND:TerminalBlock_RND_205-00235_1x05_P5.08mm_Horizontal
- JS1: footprint (none) -> joystick:C&K_THB001P
- R1: footprint (none) -> Resistor_SMD:R_0805_2012Metric_Pad1.15x1.40mm_HandSolder
Changed lines of the file:
@@
 F 0 "JS1" H 2350 1825 50  0000 C CNN
 F 1 "thb-1841844" H 2350 1734 50  0000 C CNN
-F 2 "" H 2350 1500 50  0001 C CNN
+F 2 "joystick:C&K_THB001P" H 2350 1500 50  0001 C CNN
 F 3 "" H 2350 1500 50  0001 C CNN
 	1    2350 1400
@@
 F 0 "J1" H 3880 1392 50  0000 L CNN
 F 1 "Screw_Terminal_01x05" H 3880 1301 50  0000 L CNN
-F 2 "" H 3800 1350 50  0001 C CNN
+F 2 "TerminalBlock_RND:TerminalBlock_RND_205-00235_1x05_P5.08mm_Horizontal" H 3800 1350 50  0001 C CNN
 F 3 "~" H 3800 1350 50  0001 C CNN
 	1    3800 1350
@@
 F 0 "R1" H 2868 1746 50  0000 L CNN
 F 1 "R_US" H 2868 1655 50  0000 L CNN
-F 2 "" V 2840 1690 50  0001 C CNN
+F 2 "Resistor_SMD:R_0805_2012Metric_Pad1.15x1.40mm_HandSolder" V 2840 1690 50  0001 C CNN
 F 3 "~" H 2800 1700 50  0001 C CNN
 	1    2800 1700
@@
 F 0 "H1" H 1250 796 50  0000 L CNN
 F 1 "MountingHole" H 1250 705 50  0000 L CNN
-F 2 "" H 1150 750 50  0001 C CNN
+F 2 "MountingHole:MountingHole_3.2mm_M3" H 1150 750 50  0001 C CNN
 F 3 "~" H 1150 750 50  0001 C CNN
 	1    1150 750
@@
 F 0 "H2" H 1950 796 50  0000 L CNN
 F 1 "MountingHole" H 1950 705 50  0000 L CNN
-F 2 "" H 1850 750 50  0001 C CNN
+F 2 "MountingHole:MountingHole_3.2mm_M3" H 1850 750 50  0001 C CNN
 F 3 "~" H 1850 750 50  0001 C CNN
 	1    1850 750
@@
 F 0 "H3" H 2650 796 50  0000 L CNN
 F 1 "MountingHole" H 2650 705 50  0000 L CNN
-F 2 "" H 2550 750 50  0001 C CNN
+F 2 "MountingHole:MountingHole_3.2mm_M3" H 2550 750 50  0001 C CNN
 F 3 "~" H 2550 750 50  0001 C CNN
 	1    2550 750
@@
 F 0 "H4" H 3400 796 50  0000 L CNN
 F 1 "MountingHole" H 3400 705 50  0000 L CNN
-F 2 "" H 3300 750 50  0001 C CNN
+F 2 "MountingHole:MountingHole_3.2mm_M3" H 3300 750 50  0001 C CNN
 F 3 "~" H 3300 750 50  0001 C CNN
 	1    3300 750
