File: KiCAD/comparator/comparator.kicad_pcb (KiCad board)
At the start: 2 copper layers, 71.6 x 34.5 mm, 12 parts, among them J1 Output, J2 Input, U1 TLC3704, U2 TLC3704

Commit message: saving comparator progress
Parts:
- added REF**: HP_CON_001a, Terminal_labels:HP_CON_001a, F.Cu at (130.6, 118.4)
- added REF**: HP_CON_001a, Terminal_labels:HP_CON_001a, F.Cu at (130.5, 106.0)
Other:
- board text added: "<-Inputs"
- board text added: "Outputs->"
Changed lines of the file:
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@@
   (general
     (thickness 1.6)
-    (drawings 4)
+    (drawings 6)
     (tracks 233)
     (zones 0)
-    (modules 12)
+    (modules 14)
     (nets 19)
   )
@@
     (add_net H)
   )
+  (module Terminal_labels:HP_CON_001a (layer F.Cu)
+    (at 130.6 118.425 90)
+    (fp_text reference REF** (at -13.5636 0.754 90) (layer F.SilkS) hide
+      (effects (font (size 1 1) (thickness 0.15)))
+    )
+    (fp_text value HP_CON_001a (at -13.5636 -0.246 90) (layer F.Fab)
+      (effects (font (size 1 1) (thickness 0.15)))
+    )
+    (fp_text user 5 (at 0 0 90) (layer F.SilkS)
+      (effects (font (size 1 1) (thickness 0.15)))
+    )
+    (fp_text user 8 (at 0 15.24 90) (layer F.SilkS)
+      (effects (font (size 1 1) (thickness 0.15)))
+    )
+    (fp_text user 7 (at 0 10.16 90) (layer F.SilkS)
+      (effects (font (size 1 1) (thickness 0.15)))
+    )
+    (fp_text user 6 (at 0 5.08 90) (layer F.SilkS)
+      (effects (font (size 1 1) (thickness 0.15)))
+    )
+    (fp_text user 4 (at 0 -5.08 90) (layer F.SilkS)
+      (effects (font (size 1 1) (thickness 0.15)))
+    )
+    (fp_text user 3 (at 0 -10.16 90) (layer F.SilkS)
+      (effects (font (size 1 1) (thickness 0.15)))
+    )
+    (fp_text user 2 (at 0 -15.24 90) (layer F.SilkS)
+      (effects (font (size 1 1) (thickness 0.15)))
+    )
+    (fp_text user 1 (at 0 -20.32 90) (layer F.SilkS)
+      (effects (font (size 1 1) (thickness 0.15)))
+    )
+    (fp_text user 5V (at 0 -25.4 90) (layer F.SilkS)
+      (effects (font (size 1 1) (thickness 0.15)))
+    )
+    (fp_text user GND (at 0 -30.48 90) (layer F.SilkS)
+      (effects (font (size 1 1) (thickness 0.15)))
+    )
+  )
+  (module Terminal_labels:HP_CON_001a (layer F.Cu)
+    (at 130.5 105.975 90)
+    (fp_text reference REF** (at -13.5636 0.754 90) (layer F.SilkS) hide
+      (effects (font (size 1 1) (thickness 0.15)))
+    )
+    (fp_text value HP_CON_001a (at -13.5636 -0.246 90) (layer F.Fab)
+      (effects (font (size 1 1) (thickness 0.15)))
+    )
+    (fp_text user 5 (at 0 0 90) (layer F.SilkS)
+      (effects (font (size 1 1) (thickness 0.15)))
+    )
+    (fp_text user 8 (at 0 15.24 90) (layer F.SilkS)
+      (effects (font (size 1 1) (thickness 0.15)))
+    )
+    (fp_text user 7 (at 0 10.16 90) (layer F.SilkS)
+      (effects (font (size 1 1) (thickness 0.15)))
+    )
+    (fp_text user 6 (at 0 5.08 90) (layer F.SilkS)
+      (effects (font (size 1 1) (thickness 0.15)))
+    )
+    (fp_text user 4 (at 0 -5.08 90) (layer F.SilkS)
+      (effects (font (size 1 1) (thickness 0.15)))
+    )
+    (fp_text user 3 (at 0 -10.16 90) (layer F.SilkS)
+      (effects (font (size 1 1) (thickness 0.15)))
+    )
+    (fp_text user 2 (at 0 -15.24 90) (layer F.SilkS)
+      (effects (font (size 1 1) (thickness 0.15)))
+    )
+    (fp_text user 1 (at 0 -20.32 90) (layer F.SilkS)
+      (effects (font (size 1 1) (thickness 0.15)))
+    )
+    (fp_text user 5V (at 0 -25.4 90) (layer F.SilkS)
+      (effects (font (size 1 1) (thickness 0.15)))
+    )
+    (fp_text user GND (at 0 -30.48 90) (layer F.SilkS)
+      (effects (font (size 1 1) (thickness 0.15)))
+    )
+  )
   (module MountingHole:MountingHole_3.2mm_M3 (layer F.Cu)
     (at 153.72 125)
@@
     (descr "terminal block RND 205-00240, 10 pins, pitch 5.08mm, size 50.8x8.45mm^2, drill diamater 1.1mm, pad diameter 2.1mm, see http://cdn-reichelt.de/documents/datenblatt/C151/RND_205-00232_DB_EN.pdf, script-generated using https://github.com/pointhi/kicad-footprint-generator/scripts/TerminalBlock_RND")
     (tags "THT terminal block RND 205-00240 pitch 5.08mm size 50.8x8.45mm^2 drill 1.1mm pad 2.1mm")
-    (fp_text reference J1 (at 22.86 -5.46) (layer F.SilkS)
+    (fp_text reference J1 (at 22.9 5.4) (layer F.SilkS)
       (effects (font (size 1 1) (thickness 0.15)))
     )
@@
     (fp_line (start 48.76 4.55) (end 48.76 -4.9) (layer F.CrtYd) (width 0.05))
     (fp_line (start 48.76 -4.9) (end -3.04 -4.9) (layer F.CrtYd) (width 0.05))
-    (fp_text user %R (at 22.86 -5.46) (layer F.Fab)
+    (fp_text user %R (at 22.875 5.4) (layer F.Fab)
       (effects (font (size 1 1) (thickness 0.15)))
     )
@@
     (tags "SOIC SO")
     (attr smd)
-    (fp_text reference U1 (at 0 -5.28) (layer F.SilkS)
+    (fp_text reference U1 (at -5.01 0.05) (layer F.SilkS)
       (effects (font (size 1 1) (thickness 0.15)))
     )
@@
     (tags "SOIC SO")
     (attr smd)
-    (fp_text reference U2 (at 0 -5.28) (layer F.SilkS)
+    (fp_text reference U2 (at 4.815 0.025) (layer F.SilkS)
       (effects (font (size 1 1) (thickness 0.15)))
     )
@@
     )
   )
+  (gr_text Outputs-> (at 153.675 111.8 90) (layer F.Cu)
+    (effects (font (size 2 2) (thickness 0.3)))
+  )
+  (gr_text <-Inputs (at 91.85 112.675 90) (layer F.Cu)
+    (effects (font (size 2 2) (thickness 0.3)))
+  )
   (gr_line (start 87.05 129.5) (end 87.05 95) (layer Edge.Cuts) (width 0.05))
